File: WeatherPill/WeatherPill.kicad_sch (KiCad schematic)
At the start: 64 parts, among them J1 Conn_01x02_Pin, J2 12402012E212A, J3 Conn_02x04_Odd_Even, J4 Conn_02x05_Odd_Even, J5 Conn_02x08_Odd_Even, Q1 PMOS, Q2 PMOS, SW2 SW_DPDT_x2, SW3 EVQ-P7A01P, SW4 EVQ-P7A01P, U1 USBLC6-2SC6, U2 STM32L052K8Tx, U3 sst25vf512a-33-4c-sae, U4 BU9796AMUV-E2, U5 BME280

Commit message: V2 cooking
Parts:
- removed BT1: BK-912-TR, bk-912-tr:MPD_BK-912-TR, symbol BK-912-TR:BK-912-TR
- removed D2, D3: LTST-C190GKT, green led:LEDM1608X80, symbol green led:LTST-C190GKT
- removed H1, H2, H3, H4: MountingHole, MountingHole:MountingHole_3.2mm_M3_DIN965, symbol Mechanical:MountingHole
- removed J1: Conn_01x02_Pin, Connector_PinHeader_2.54mm:PinHeader_1x02_P2.54mm_Vertical, symbol Connector:Conn_01x02_Pin
- removed J2: 12402012E212A, USB12402012E212A:AMPHENOL_12402012E212A, symbol usb conn:12402012E212A
- removed J3: Conn_02x04_Odd_Even, Connector_PinSocket_2.54mm:PinSocket_2x04_P2.54mm_Vertical, symbol Connector_Generic:Conn_02x04_Odd_Even
- removed J4: Conn_02x05_Odd_Even, Connector_PinHeader_2.54mm:PinHeader_2x05_P2.54mm_Vertical, symbol Connector_Generic:Conn_02x05_Odd_Even
- removed J5: Conn_02x08_Odd_Even, Connector_PinHeader_2.54mm:PinHeader_2x08_P2.54mm_Vertical, symbol Connector_Generic:Conn_02x08_Odd_Even
- removed JP1: SolderJumper_3_Open, Jumper:SolderJumper-3_P1.3mm_Open_Pad1.0x1.5mm_NumberLabels, symbol Jumper:SolderJumper_3_Open
- removed Q1, Q2: PMOS, Package_TO_SOT_SMD:SOT-323_SC-70_Handsoldering, symbol Simulation_SPICE:PMOS
- removed R21, R22, R23, R24, R25, R26, R27, R28: 0R, Capacitor_SMD:C_0603_1608Metric_Pad1.08x0.95mm_HandSolder, symbol Device:R
- removed R30, R31: 240R, Resistor_SMD:R_0603_1608Metric_Pad0.98x0.95mm_HandSolder, symbol Device:R_Small
- removed SW2: SW_DPDT_x2, dpdt_switch:450404015514, symbol Switch:SW_DPDT_x2
- removed U1: USBLC6-2SC6, Package_TO_SOT_SMD:SOT-23-6, symbol Power_Protection:USBLC6-2SC6
- removed U2: STM32L052K8Tx, Package_QFP:LQFP-32_7x7mm_P0.8mm, symbol MCU_ST_STM32L0:STM32L052K8Tx
- removed U3: sst25vf512a-33-4c-sae, sst25vf5:SOIC8_SA_SST_MCH, symbol sst25vf512a-33-4c-sae:sst25vf512a-33-4c-sae
- removed U4: BU9796AMUV-E2, lcd driver:VQFN024V4040_ROM, symbol lcd driver:BU9796AMUV-E2
- added BT1: 1056, batt12mm:BAT_1056, symbol battery 12 mm:1056
- added C11, C12: 1uf, LED_SMD:LED_0402_1005Metric_Pad0.77x0.64mm_HandSolder, symbol Device:C
- added C13, C9: 100nF, LED_SMD:LED_0402_1005Metric_Pad0.77x0.64mm_HandSolder, symbol Device:C
- added J1: Conn_ARM_SWD_TagConnect_TC2030-NL, Connector:Tag-Connect_TC2030-IDC-NL_2x03_P1.27mm_Vertical, symbol Connector:Conn_ARM_SWD_TagConnect_TC2030-NL
- added J2: USB4105-GF-A, usb conn atomic:GCT_USB4105-GF-A, symbol usb-4105:USB4105-GF-A
- added R30, R31, R32, R33, R34, R35, R36, R37, R38: 0R, Resistor_SMD:R_0201_0603Metric_Pad0.64x0.40mm_HandSolder, symbol Device:R
- added R4: 5.1k, Resistor_SMD:R_0201_0603Metric_Pad0.64x0.40mm_HandSolder, symbol Device:R
- added SW1: CUS-12TB, CUS-12TB_NDC, symbol petite switch:CUS-12TB
- added TP1: VBATT, TestPoint:TestPoint_Pad_D1.5mm, symbol Connector:TestPoint
- added TP2: GND, TestPoint:TestPoint_Pad_D1.5mm, symbol Connector:TestPoint
- added U1: USBLC6-2P6, Package_TO_SOT_SMD:SOT-666, symbol Power_Protection:USBLC6-2P6
- added U2: ~, Package_DFN_QFN:HVQFN-32-1EP_5x5mm_P0.5mm_EP3.1x3.1mm, symbol New_Library:PCA8561
- added U3: SHT4x, Sensor_Humidity:Sensirion_DFN-4_1.5x1.5mm_P0.8mm_SHT4x_NoCentralPad, symbol Sensor_Humidity:SHT4x
- added U4: TPS22916CYFPR, loadswitch:YFP0004ABAB, symbol loadswitch:TPS22916CYFPR
- added U6: HDC2010YPAR, HDC:BGA6C100X50P2X3_HDC2010YPAR, symbol HD2010:HDC2010YPAR
- added U7: BMP581, bmp581:QFN10_BMP581_BOS-M, symbol bmp581:BMP581
- added U8: STM32L072KZUx, Package_DFN_QFN:QFN-32-1EP_5x5mm_P0.5mm_EP3.45x3.45mm, symbol MCU_ST_STM32L0:STM32L072KZUx
- C1, C10, C2, C3, C4, C5, C6, C7: footprint Capacitor_SMD:C_0603_1608Metric_Pad1.08x0.95mm_HandSolder -> LED_SMD:LED_0402_1005Metric_Pad0.77x0.64mm_HandSolder
- C8: value 0.1uF -> 100nF; footprint Capacitor_SMD:C_0603_1608Metric_Pad1.08x0.95mm_HandSolder -> LED_SMD:LED_0402_1005Metric_Pad0.77x0.64mm_HandSolder
- L1: footprint Library:lcd_ebay -> led7segment:INND-SS30
- R1, R11, R12, R13, R14, R15, R16, R17, R18, R19, R20, R5, R6, R7, R8: footprint Capacitor_SMD:C_0603_1608Metric_Pad1.08x0.95mm_HandSolder -> Resistor_SMD:R_0201_0603Metric_Pad0.64x0.40mm_HandSolder
- R10, R9: value 1M -> 0R; footprint Capacitor_SMD:C_0603_1608Metric_Pad1.08x0.95mm_HandSolder -> Resistor_SMD:R_0201_0603Metric_Pad0.64x0.40mm_HandSolder
- R2: value 1M -> 1K; footprint Capacitor_SMD:C_0603_1608Metric_Pad1.08x0.95mm_HandSolder -> Resistor_SMD:R_0201_0603Metric_Pad0.64x0.40mm_HandSolder
- R29: value 240R -> 470R; footprint Resistor_SMD:R_0603_1608Metric_Pad0.98x0.95mm_HandSolder -> Resistor_SMD:R_0201_0603Metric_Pad0.64x0.40mm_HandSolder
- R3: value 0R -> 5.1k; footprint Capacitor_SMD:C_0603_1608Metric_Pad1.08x0.95mm_HandSolder -> Resistor_SMD:R_0201_0603Metric_Pad0.64x0.40mm_HandSolder
Connections:
- net BOOT is gone; now on net BTN_2: R2.1
- net CONTROL_ZONE_2 is gone; now on net GND: R9.2
- net SCK_BME280 is gone; now on an unnamed net: U5.4 (SCK)
- net SDI_BME280 is gone; now on an unnamed net: U5.3 (SDI)
- net V_BUS_DISPLAY is gone; now on net V_BUS_3V: C10.1
- net V_BUS_ZONE_2 is gone; now on net V_BUS_ZONE_1: R11.2, R12.2
- net BTN_1: now also U8.7 (PA1)
- net CONTROL_ZONE_1: now also U4.B2 (ON), U8.29 (PB7); no longer R10.2
- net CS_1: now also R18.2, U8.9 (PA3)
- net CS_2: now also R37.2, U8.10 (PA4)
- net GND: now also C4.1, R3.1, SW4.1, BT1.N, C11.2, C12.2, C13.2, C9.1, J1.5 (GND), J2.A1_B12 (GND), J2.B1_A12 (GND__1), J2.SH1 (SHELL_GND), J2.SH2 (SHELL_GND__1), J2.SH3 (SHELL_GND__2), J2.SH4 (SHELL_GND__3), R32.2, R4.2, TP2.1, U1.2 (GND), U3.4 (VSS), U4.B1 (GND), U6.C1 (GND), U7.3 (VSS), U7.8 (VSS), U7.9 (VSS), U8.16 (VSS), U8.31 (VSS), U8.33 (VSS), U8.4 (VSSA); no longer R1.2, R15.2, R16.2, R17.2, R18.1, R19.2, R3.2, R5.2, SW3.2*, SW4.2, SW4.2*
- net NRST: now also J1.3 (~{RESET}), U8.3 (NRST)
- net SCK_1: now also R16.2, R35.2, U8.11 (PA5)
- net SCL_1: now also R1.2, R30.2, U8.19 (PA9)
- net SDA_1: now also R10.2, R31.2, U8.20 (PA10)
- net SDI_1: now also R17.2, R36.2, U8.12 (PA6)
- net SDO_1: now also R14.2, R34.2, U8.13 (PA7)
- net SWCLK: now also J1.4 (SWCLK), U8.25 (PA14)
- net SWDIO: now also J1.2 (SWDIO), U8.23 (PA13)
- net SWO: now also J1.6 (SWO)
- net USB_D+: now also J2.A6 (DP1), J2.B6 (DP2), U1.1 (I/O1), U1.6 (I/O1), U8.21 (PA11); no longer C4.1
- net USB_D-: now also J2.A7 (DN1), J2.B7 (DN2), U1.3 (I/O2), U1.4 (I/O2), U8.22 (PA12); no longer C4.2
- net V_BUS_3V: now also R15.1, C11.1, J1.1 (VCC), SW1.3, U4.A2 (VIN), U8.17 (VDD), U8.32 (VDD), U8.5 (VDDA); no longer R10.1, R9.1
- net V_BUS_ZONE_1: now also C4.2, R15.2, C12.1, C13.1, C9.2, U3.3 (VDD), U4.A1 (VOUT), U6.A1 (VDD), U7.1 (VDDIO), U7.10 (VDD); no longer R14.1
- net at R1.1: now also U3.2 (SCL)
- net at R20.1: now also U8.26 (PB4)
- net at R6.1: now also U8.14 (PB0)
- net at C5.2, R8.1: now also SW3.1; no longer SW3.1*
- net at R7.1: now also U8.15 (PB1)
- net at C6.2, R13.1: now also SW4.2; no longer SW4.1*
- net at R2.2: now also U8.30 (BOOT0)
- net at L1.10: no longer L1.9
- net at L1.7: no longer L1.8
- net V_USB: now reaches R19.1
- net V_USB: now also J2.A4_B9 (VBUS), J2.B4_A9 (VBUS__1), U1.5 (VBUS), U8.24 (VDD_USB)
- net CS_BME280: no longer names the net of U5.2 (CSB)
- net CS_BME280: now also R18.1
- net LED0: no longer names the net of R29.1
- net LED0: now also U8.28 (PB6)
- net SDO_BME280: no longer names the net of U5.5 (SDO)
- net SDO_BME280: now also R14.1
- new net: BT1.P, SW1.2, TP1.1
- new net: R10.1, U3.1 (SDA)
- new net: R9.1, U8.27 (PB5)
- new net: R31.1, U6.A2 (SDA)
- new net: R32.1, U6.B1 (ADDR)
- new net: R30.1, U6.B2 (SCL)
- new net: R33.2, U6.C2 (DRDY/INT)
- new net: J2.B5 (CC2), R3.2
- new net: R5.2, U8.8 (PA2)
- new net: R35.1, U7.2 (SCK)
- new net: R34.1, U7.5 (SDO)
- new net: R36.1, U7.4 (SDI)
- new net: J2.A5 (CC1), R4.1
- new net: R38.1, U7.7 (INT)
- new net: R37.1, U7.6 (CSB)
- new net HDC_DRDY: R33.1, U8.18 (PA8)
- no-connect marks 1 -> 10
Other:
- note added: "SENSOR 1"
- note removed: "DISPLAY"
- note removed: "MEMORY"
- note removed: "SENSOR 3"
- moved on the sheet: C1, C2, C3, C5, C6, C7, D1, R11, R12, R13, R2, R20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

Commit message: rev 2 sent
Parts:
- removed R5: 0R, Resistor_SMD:R_0201_0603Metric_Pad0.64x0.40mm_HandSolder, symbol Device:R
- added C15, C16: 100nF, LED_SMD:LED_0402_1005Metric_Pad0.77x0.64mm_HandSolder, symbol Device:C
- added R21, R22, R23, R24: 0R, Resistor_SMD:R_0201_0603Metric_Pad0.64x0.40mm_HandSolder, symbol Device:R
- added TP3, TP4: TestPoint, symbol Connector:TestPoint
Connections:
- net BTN_1: now also U8.6 (PA0); no longer U8.7 (PA1)
- net BTN_2: now also U8.7 (PA1); no longer R2.1
- net GND: now also R2.1, U2.4 (VSS), C15.2, C16.2, R21.2, R22.2, R23.2, R24.2
- net SCL_1: now also U2.8 (SCL)
- net SDA_1: now also U2.9 (_CE)
- net V_BUS_ZONE_1: now also U2.2 (VLCD), U2.3 (VDD), C15.1, C16.1
- net SEG0: now reaches L1.1
- net SEG0: now also U2.12 (SEG0)
- net COM0: now reaches L1.10
- net COM0: now also U2.30 (COM0)
- net SEG1: now reaches L1.2
- net SEG1: now also U2.13 (SEG1)
- net SEG2: now reaches L1.3
- net SEG2: now also U2.14 (SEG2)
- net SEG3: now reaches L1.4
- net SEG3: now also U2.15 (SEG3)
- net SEG4: now reaches L1.5
- net SEG4: now also U2.16 (SEG4)
- net SEG5: now reaches L1.6
- net SEG5: now also U2.17 (SEG5)
- net COM3: now reaches L1.7
- net COM3: now also U2.1 (COM3)
- net COM2: now reaches L1.8
- net COM2: now also U2.32 (COM2)
- net COM1: now reaches L1.9
- net COM1: now also U2.31 (COM1)
- net at SW4.2: now also C6.2, R13.1
- net at U2.10 (PORE): now also R24.1
- net ~{DISP_RST}: now reaches U2.5 (_RST)
- net ~{DISP_RST}: now also U8.8 (PA2)
- net at U2.6 (SDIO): now also TP3.1
- net at U2.7 (CLK): now also R21.1
- new net: R23.1, U2.11 (nc)
- new net: TP4.1, U2.9 (_CE)
- new net: R22.1, U2.6 (SDIO)
